Commit message: Enable collision for ocean1 left and right end effectors

File: urdf_models/ocean1/ocean1.urdf (robot description, URDF)
Before this commit: robot ocean1, 21 links, 20 joints
Links:
- link endEffector_left: geometry collision box size=0.1 0.1 0.1; visual box size=0.1 0.1 0.1
- link endEffector_right: geometry collision box size=0.1 0.1 0.1; visual box size=0.1 0.1 0.1

Commit message: Update end effector visuals to ocean1 hands rather than box

File: urdf_models/ocean1/ocean1.urdf (robot description, URDF)
Before this commit: robot ocean1, 21 links, 20 joints
Links:
- link endEffector_left: geometry collision box size=0.1 0.1 0.1; visual mesh filename=ocean1_graphics/HandO2.obj
- link endEffector_right: geometry collision box size=0.1 0.1 0.1; visual mesh filename=ocean1_graphics/HandO2.obj
